File: fonte.brd (EAGLE design)
At the start: 100 x 81.3 mm, 19 parts, among them T1 BP103

Commit message: Add files via upload
Parts:
- removed T1: BP103, opto-trans-siemens:BP103
- removed TR1: (no value), inductor-neosid:U15
- added T2: BC337, transistor:TO92
- moved D5 41.0 mm to (34.3, 17.8)
- moved R2 29.3 mm to (74.9, 31.8), turned to 270 degrees
- moved D6 21.7 mm to (86.4, 33.0)
- moved R1 20.3 mm to (10.2, 24.1)
- moved R3 19.1 mm to (48.3, 54.6)
- moved D3 16.6 mm to (27.9, 52.1)
- moved C1 15.5 mm to (88.9, 53.3)
- moved R6 14.2 mm to (71.1, 52.1), turned to 270 degrees
- moved R4 13.0 mm to (36.8, 45.7)
- moved D4 12.0 mm to (19.1, 66.0)
- moved D2 10.8 mm to (36.8, 71.1)
- moved R5 9.92 mm to (20.3, 57.1)
- moved JP1 8.98 mm to (3.81, 62.2), turned to 270 degrees
- moved R13 8.13 mm to (49.5, 45.7)
- moved JP2 6.48 mm to (95.2, 40.6)
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Connections:
- removed net N$10: JP1.2, TR1.2
- removed net N$11: JP1.1, TR1.1
- removed net N$12: D2.A, D4.C, TR1.3
- new net N$4: D2.A, D4.C, JP1.1
- net 1: now also T2.1; no longer T1.E
- net N$13: now also T2.3; no longer T1.C
- net N$2: now also JP1.2; no longer TR1.4
- net N$6: now also T2.2; no longer T1.B
Routing:
- net 0: track 138.6 -> 189.7 mm
- net N$2: track 23.4 -> 68.2 mm
- net N$12: track 44.4 -> 0.00 mm
- net N$1: track 7.93 -> 40.5 mm
- net N$4: track 0.00 -> 32.4 mm
- net N$7: track 8.89 -> 37.0 mm
- net N$6: track 41.8 -> 67.0 mm
- net N$3: track 6.22 -> 28.1 mm
- net N$13: track 141.1 -> 156.7 mm
- net N$5: track 58.2 -> 43.2 mm
- net N$11: track 10.4 -> 0.00 mm
- net N$10: track 9.32 -> 0.00 mm
- net 1: track 83.0 -> 75.4 mm
