File: fonte.sch (EAGLE design)
At the start: 19 parts, among them T1 BP103

Commit message: Add files via upload
Parts:
- removed T1: BP103, opto-trans-siemens:BP103
- removed TR1: (no value), inductor-neosid:U15-TRANSFORMER
- added T2: BC337, transistor:BC337
Connections:
- removed net N$10: JP1.2, TR1.2
- removed net N$11: JP1.1, TR1.1
- removed net N$12: D2.A, D4.C, TR1.3
- new net N$4: D2.A, D4.C, JP1.1
- net 1: now also T2.E; no longer T1.E
- net N$13: now also T2.C; no longer T1.C
- net N$2: now also JP1.2; no longer TR1.4
- net N$6: now also T2.B; no longer T1.B
Changed lines of the file:
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@@
 <part name="C2" library="capacitor-wima" library_urn="urn:adsk.eagle:library:116" deviceset="C" device="5/3" package3d_urn="urn:adsk.eagle:package:5433/1"/>
 <part name="R1" library="piher" library_urn="urn:adsk.eagle:library:324" deviceset="PC16S" device="" package3d_urn="urn:adsk.eagle:package:22243/1"/>
-<part name="TR1" library="inductor-neosid" library_urn="urn:adsk.eagle:library:241" deviceset="U15" device="-TRANSFORMER" package3d_urn="urn:adsk.eagle:package:14678/1"/>
 <part name="JP1" library="pinhead" library_urn="urn:adsk.eagle:library:325" deviceset="PINHD-1X2" device="" package3d_urn="urn:adsk.eagle:package:22435/2"/>
 <part name="JP2" library="pinhead" library_urn="urn:adsk.eagle:library:325" deviceset="PINHD-1X2" device="" package3d_urn="urn:adsk.eagle:package:22435/2"/>
 <part name="C1" library="capacitor-wima" library_urn="urn:adsk.eagle:library:116" deviceset="C" device="5/3" package3d_urn="urn:adsk.eagle:package:5433/1"/>
-<part name="T1" library="opto-trans-siemens" library_urn="urn:adsk.eagle:library:317" deviceset="BP103" device="" package3d_urn="urn:adsk.eagle:package:21787/1"/>
 <part name="R2" library="rcl" library_urn="urn:adsk.eagle:library:334" deviceset="R-EU_" device="0204/7" package3d_urn="urn:adsk.eagle:package:23498/1"/>
 <part name="R3" library="rcl" library_urn="urn:adsk.eagle:library:334" deviceset="R-EU_" device="0204/7" package3d_urn="urn:adsk.eagle:package:23498/1"/>
@@
 <part name="R13" library="rcl" library_urn="urn:adsk.eagle:library:334" deviceset="R-EU_" device="0204/7" package3d_urn="urn:adsk.eagle:package:23498/1"/>
 <part name="D6" library="display-hp" library_urn="urn:adsk.eagle:library:212" deviceset="HLMP6" device="" package3d_urn="urn:adsk.eagle:package:12992/1"/>
+<part name="T2" library="transistor" library_urn="urn:adsk.eagle:library:402" deviceset="BC337" device="" package3d_urn="urn:adsk.eagle:package:29893/2"/>
 </parts>
 <sheets>
@@
 <attribute name="VALUE" x="143.51" y="56.134" size="1.778" layer="96" rot="R90"/>
 </instance>
-<instance part="TR1" gate="G$1" x="27.94" y="58.42" smashed="yes" rot="R90">
-<attribute name="NAME" x="24.584" y="55.88" size="1.778" layer="95" rot="R90"/>
-<attribute name="VALUE" x="33.02" y="55.626" size="1.778" layer="96" rot="R90"/>
-</instance>
 <instance part="JP1" gate="G$1" x="0" y="60.96" rot="R180"/>
 <instance part="JP2" gate="G$1" x="226.06" y="45.72"/>
@@
 <attribute name="VALUE" x="209.296" y="50.419" size="1.778" layer="96" rot="R180"/>
 </instance>
-<instance part="T1" gate="1" x="170.18" y="63.5"/>
 <instance part="R2" gate="G$1" x="114.3" y="68.58" rot="R90"/>
 <instance part="R3" gate="G$1" x="114.3" y="48.26" rot="R90"/>
@@
 <instance part="R13" gate="G$1" x="198.12" y="50.8" rot="R90"/>
 <instance part="D6" gate="A" x="198.12" y="63.5"/>
+<instance part="T2" gate="G$1" x="170.18" y="63.5"/>
 </instances>
 <busses>
@@
 <pinref part="R4" gate="G$1" pin="1"/>
 <junction x="132.08" y="66.04"/>
-</segment>
-</net>
-<net name="N$10" class="0">
-<segment>
-<wire x1="5.08" y1="68.58" x2="25.4" y2="68.58" width="0.1524" layer="91"/>
-<pinref part="TR1" gate="G$1" pin="2"/>
-<wire x1="25.4" y1="68.58" x2="25.4" y2="66.04" width="0.1524" layer="91"/>
-<pinref part="JP1" gate="G$1" pin="2"/>
-<wire x1="2.54" y1="60.96" x2="5.08" y2="60.96" width="0.1524" layer="91"/>
-<wire x1="5.08" y1="60.96" x2="5.08" y2="68.58" width="0.1524" layer="91"/>
-</segment>
-</net>
-<net name="N$11" class="0">
-<segment>
-<wire x1="5.08" y1="48.26" x2="25.4" y2="48.26" width="0.1524" layer="91"/>
-<pinref part="TR1" gate="G$1" pin="1"/>
-<wire x1="25.4" y1="48.26" x2="25.4" y2="53.34" width="0.1524" layer="91"/>
-<pinref part="JP1" gate="G$1" pin="1"/>
-<wire x1="2.54" y1="58.42" x2="5.08" y2="58.42" width="0.1524" layer="91"/>
-<wire x1="5.08" y1="58.42" x2="5.08" y2="48.26" width="0.1524" layer="91"/>
-</segment>
-</net>
-<net name="N$2" class="0">
-<segment>
-<wire x1="45.72" y1="68.58" x2="45.72" y2="81.28" width="0.1524" layer="91"/>
-<pinref part="D1" gate="G$1" pin="A"/>
-<wire x1="45.72" y1="81.28" x2="63.5" y2="81.28" width="0.1524" layer="91"/>
-<pinref part="D3" gate="G$1" pin="C"/>
-<wire x1="63.5" y1="81.28" x2="71.12" y2="81.28" width="0.1524" layer="91"/>
-<wire x1="71.12" y1="50.8" x2="63.5" y2="50.8" width="0.1524" layer="91"/>
-<wire x1="63.5" y1="50.8" x2="63.5" y2="81.28" width="0.1524" layer="91"/>
-<junction x="63.5" y="81.28"/>
-<pinref part="TR1" gate="G$1" pin="4"/>
-<wire x1="45.72" y1="68.58" x2="30.48" y2="68.58" width="0.1524" layer="91"/>
-<wire x1="30.48" y1="68.58" x2="30.48" y2="66.04" width="0.1524" layer="91"/>
-</segment>
-</net>
-<net name="N$12" class="0">
-<segment>
-<wire x1="45.72" y1="48.26" x2="45.72" y2="35.56" width="0.1524" layer="91"/>
-<pinref part="D4" gate="G$1" pin="C"/>
-<wire x1="45.72" y1="35.56" x2="55.88" y2="35.56" width="0.1524" layer="91"/>
-<wire x1="55.88" y1="35.56" x2="73.66" y2="35.56" width="0.1524" layer="91"/>
-<wire x1="78.74" y1="66.04" x2="76.962" y2="66.04" width="0.1524" layer="91"/>
-<wire x1="76.962" y1="66.04" x2="55.88" y2="66.04" width="0.1524" layer="91"/>
-<wire x1="55.88" y1="66.04" x2="55.88" y2="35.56" width="0.1524" layer="91"/>
-<junction x="55.88" y="35.56"/>
-<pinref part="D2" gate="G$1" pin="A"/>
-<junction x="76.962" y="66.04"/>
-<pinref part="TR1" gate="G$1" pin="3"/>
-<wire x1="45.72" y1="48.26" x2="30.48" y2="48.26" width="0.1524" layer="91"/>
-<wire x1="30.48" y1="48.26" x2="30.48" y2="53.34" width="0.1524" layer="91"/>
 </segment>
 </net>
@@
 <junction x="114.3" y="81.28"/>
 <pinref part="C2" gate="G$1" pin="1"/>
-<pinref part="T1" gate="1" pin="C"/>
 <pinref part="R2" gate="G$1" pin="2"/>
 <pinref part="R4" gate="G$1" pin="2"/>
+<pinref part="T2" gate="G$1" pin="C"/>
 </segment>
 </net>
@@
 <wire x1="152.4" y1="58.42" x2="149.86" y2="58.42" width="0.1524" layer="91"/>
 <wire x1="162.56" y1="63.5" x2="167.64" y2="63.5" width="0.1524" layer="91"/>
-<pinref part="T1" gate="1" pin="B"/>
+<pinref part="T2" gate="G$1" pin="B"/>
 </segment>
 </net>
@@
 <wire x1="223.52" y1="55.88" x2="223.52" y2="48.26" width="0.1524" layer="91"/>
 <junction x="210.82" y="55.88"/>
-<pinref part="T1" gate="1" pin="E"/>
 <pinref part="R6" gate="G$1" pin="2"/>
 <pinref part="D6" gate="A" pin="A"/>
+<pinref part="T2" gate="G$1" pin="E"/>
 </segment>
 </net>
@@
 </segment>
 </net>
+<net name="N$2" class="0">
+<segment>
+<wire x1="5.08" y1="60.96" x2="5.08" y2="68.58" width="0.1524" layer="91"/>
+<pinref part="JP1" gate="G$1" pin="2"/>
+<wire x1="2.54" y1="60.96" x2="5.08" y2="60.96" width="0.1524" layer="91"/>
+<wire x1="5.08" y1="68.58" x2="45.72" y2="68.58" width="0.1524" layer="91"/>
+<wire x1="45.72" y1="68.58" x2="45.72" y2="81.28" width="0.1524" layer="91"/>
+<pinref part="D1" gate="G$1" pin="A"/>
+<wire x1="45.72" y1="81.28" x2="63.5" y2="81.28" width="0.1524" layer="91"/>
+<pinref part="D3" gate="G$1" pin="C"/>
+<wire x1="63.5" y1="81.28" x2="71.12" y2="81.28" width="0.1524" layer="91"/>
+<wire x1="71.12" y1="50.8" x2="63.5" y2="50.8" width="0.1524" layer="91"/>
+<wire x1="63.5" y1="50.8" x2="63.5" y2="81.28" width="0.1524" layer="91"/>
+<junction x="63.5" y="81.28"/>
+</segment>
+</net>
+<net name="N$4" class="0">
+<segment>
+<pinref part="JP1" gate="G$1" pin="1"/>
+<wire x1="2.54" y1="58.42" x2="5.08" y2="58.42" width="0.1524" layer="91"/>
+<wire x1="5.08" y1="58.42" x2="5.08" y2="48.26" width="0.1524" layer="91"/>
+<wire x1="5.08" y1="48.26" x2="45.72" y2="48.26" width="0.1524" layer="91"/>
+<wire x1="45.72" y1="48.26" x2="45.72" y2="35.56" width="0.1524" layer="91"/>
+<pinref part="D4" gate="G$1" pin="C"/>
+<wire x1="45.72" y1="35.56" x2="55.88" y2="35.56" width="0.1524" layer="91"/>
+<wire x1="55.88" y1="35.56" x2="73.66" y2="35.56" width="0.1524" layer="91"/>
+<wire x1="78.74" y1="66.04" x2="76.962" y2="66.04" width="0.1524" layer="91"/>
+<wire x1="76.962" y1="66.04" x2="55.88" y2="66.04" width="0.1524" layer="91"/>
+<wire x1="55.88" y1="66.04" x2="55.88" y2="35.56" width="0.1524" layer="91"/>
+<junction x="55.88" y="35.56"/>
+<pinref part="D2" gate="G$1" pin="A"/>
+<junction x="76.962" y="66.04"/>
+</segment>
+</net>
